File: kicad/amp/amp.kicad_sch (KiCad schematic)
At the start: 13 parts, among them J1 Conn_01x02_Socket, J2 Conn_01x02_Socket, J3 Conn_01x02_Socket, U1 LM386

Commit message: USB PIO now works and can control via PC or direct MIDI device :)
Other:
- note added: "use same footprint 96mm square (or what ever it is) put some labels on the headers find the right footprints to match film caps"
